Commit message: Add new packages to catkin_ws/src

File: urdf_models/urdf/part_viewer.urdf (robot description, URDF)
Before this commit: robot irb1400, 1 links, 0 joints
Links:
- link link4: geometry collision mesh filename=package://urdf_models/meshes/link4.STL; visual mesh filename=package://urdf_models/meshes/link4.STL

Commit message: Large commit after Hokudai

File: urdf_models/urdf/part_viewer.urdf (robot description, URDF)
Before this commit: robot irb1400, 1 links, 0 joints
Links:
- link link4: geometry collision mesh filename=package://denso_ve026a/meshes/l6.stl; visual mesh filename=package://denso_ve026a/meshes/l6.stl
